File: keyboard_vero2.sch (KiCad schematic (older format))
At the start: 85 parts, among them J1 Conn_01x15_Male, SW0 SW_Push_45deg, SW1 SW_Push_45deg, SW10 SW_Push_45deg, SW11 SW_Push_45deg, SW12 SW_Push_45deg, SW13 SW_Push_45deg, SW14 SW_Push_45deg, SW15 SW_Push_45deg, SW16 SW_Push_45deg, SW17 SW_Push_45deg, SW18 SW_Push_45deg, SW19 SW_Push_45deg, SW2 SW_Push_45deg, SW20 SW_Push_45deg, SW21 SW_Push_45deg, SW22 SW_Push_45deg, SW23 SW_Push_45deg, SW24 SW_Push_45deg, SW25 SW_Push_45deg, SW26 SW_Push_45deg, SW27 SW_Push_45deg, SW28 SW_Push_45deg, SW29 SW_Push_45deg, SW3 SW_Push_45deg, SW30 SW_Push_45deg, SW31 SW_Push_45deg, SW32 SW_Push_45deg, SW33 SW_Push_45deg, SW34 SW_Push_45deg, SW35 SW_Push_45deg, SW36 SW_Push_45deg, SW37 SW_Push_45deg, SW38 SW_Push_45deg, SW39 SW_Push_45deg, SW4 SW_Push_45deg, SW40 SW_Push_45deg, SW41 SW_Push_45deg, SW42 SW_Push_45deg, SW43 SW_Push_45deg, SW44 SW_Push_45deg, SW45 SW_Push_45deg, SW46 SW_Push_45deg, SW47 SW_Push_45deg, SW48 SW_Push_45deg, SW49 SW_Push_45deg, SW5 SW_Push_45deg, SW50 SW_Push_45deg, SW51 SW_Push_45deg, SW52 SW_Push_45deg, SW53 SW_Push_45deg, SW54 SW_Push_45deg, SW55 SW_Push_45deg, SW56 SW_Push_45deg, SW57 SW_Push_45deg, SW58 SW_Push_45deg, SW59 SW_Push_45deg, SW6 SW_Push_45deg, SW60 SW_Push_45deg, SW61 SW_Push_45deg, SW62 SW_Push_45deg, SW63 SW_Push_45deg, SW7 SW_Push_45deg, SW8 SW_Push_45deg, SW9 SW_Push_45deg, U1 74LS138, U2 74LS374

Commit message: Updated schematic to match final build; created BOM
Parts:
- D1: renamed from R9; footprint Resistor_THT:R_Axial_DIN0204_L3.6mm_D1.6mm_P7.62mm_Horizontal -> Diode_THT:D_DO-35_SOD27_P7.62mm_Horizontal; symbol Device:R_Small -> Diode:1N4007
- D2: renamed from R10; footprint Resistor_THT:R_Axial_DIN0204_L3.6mm_D1.6mm_P7.62mm_Horizontal -> Diode_THT:D_DO-35_SOD27_P7.62mm_Horizontal; symbol Device:R_Small -> Diode:1N4007
- D3: renamed from R11; footprint Resistor_THT:R_Axial_DIN0204_L3.6mm_D1.6mm_P7.62mm_Horizontal -> Diode_THT:D_DO-35_SOD27_P7.62mm_Horizontal; symbol Device:R_Small -> Diode:1N4007
- D4: renamed from R12; footprint Resistor_THT:R_Axial_DIN0204_L3.6mm_D1.6mm_P7.62mm_Horizontal -> Diode_THT:D_DO-35_SOD27_P7.62mm_Horizontal; symbol Device:R_Small -> Diode:1N4007
- D5: renamed from R13; footprint Resistor_THT:R_Axial_DIN0204_L3.6mm_D1.6mm_P7.62mm_Horizontal -> Diode_THT:D_DO-35_SOD27_P7.62mm_Horizontal; symbol Device:R_Small -> Diode:1N4007
- D6: renamed from R14; footprint Resistor_THT:R_Axial_DIN0204_L3.6mm_D1.6mm_P7.62mm_Horizontal -> Diode_THT:D_DO-35_SOD27_P7.62mm_Horizontal; symbol Device:R_Small -> Diode:1N4007
- D7: renamed from R15; footprint Resistor_THT:R_Axial_DIN0204_L3.6mm_D1.6mm_P7.62mm_Horizontal -> Diode_THT:D_DO-35_SOD27_P7.62mm_Horizontal; symbol Device:R_Small -> Diode:1N4007
- D8: renamed from R16; footprint Resistor_THT:R_Axial_DIN0204_L3.6mm_D1.6mm_P7.62mm_Horizontal -> Diode_THT:D_DO-35_SOD27_P7.62mm_Horizontal; symbol Device:R_Small -> Diode:1N4007
Connections:
- net at SW0.2, SW1.2, SW2.2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: now also D1.2 (A); no longer D1.1
- net at SW10.2, SW11.2, SW12.2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: now also D2.2 (A); no longer D2.1
- net at SW16.2, SW17.2, SW18.2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: now also D3.2 (A); no longer D3.1
- net at SW24.2, SW25.2, SW26.2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: now also D4.2 (A); no longer D4.1
- net at SW32.2, SW33.2, SW34.2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: now also D5.2 (A); no longer D5.1
- net at SW40.2, SW41.2, SW42.2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: now also D6.2 (A); no longer D6.1
- net at SW48.2, SW49.2, SW50.2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: now also D7.2 (A); no longer D7.1
- net at SW56.2, SW57.2, SW58.2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: now also D8.2 (A); no longer D8.1
- net at U1.10 (O5): now also D3.1 (K); no longer D3.2
- net at U1.11 (O4): now also D4.1 (K); no longer D4.2
- net at U1.12 (O3): now also D5.1 (K); no longer D5.2
- net at U1.13 (O2): now also D6.1 (K); no longer D6.2
- net at U1.14 (O1): now also D7.1 (K); no longer D7.2
- net at U1.15 (O0): now also D8.1 (K); no longer D8.2
- net at U1.7 (O7): now also D1.1 (K); no longer D1.2
- net at U1.9 (O6): now also D2.1 (K); no longer D2.2
Other:
- note added: "08/06/2020"
- note added: "Homebrew Keyboard with Parallel Interface"

Commit message: Unlink ~OE from LS138's enable input
Connections:
- net GND: now also U1.5 (E2)
- net OE renamed ~OE
- net ~OE: no longer U1.5 (E2)
Changed lines of the file:
@@
 PHI
 Text Label 3850 2700 0    50   ~ 0
-OE
+~OE
 Wire Wire Line
 	5550 3350 5500 3350
@@
 Wire Wire Line
 	5500 3150 5550 3150
-Wire Wire Line
-	5200 3250 5550 3250
 $Comp
 L Connector:Conn_01x15_Male J1
@@
 	3750 2000 3750 2300
 Wire Wire Line
-	5200 3250 5200 5250
-Wire Wire Line
 	3400 3700 3950 3700
 Wire Wire Line
@@
 Wire Wire Line
 	3400 2700 5200 2700
-Wire Wire Line
-	5200 2700 5200 3250
-Connection ~ 5200 3250
 Wire Wire Line
 	5100 2900 5100 5150
@@
 Wire Wire Line
 	6600 3950 7150 3950
+Text Notes 7400 7500 0    69   Italic 14
+Homebrew Keyboard with Parallel Interface
+Text Notes 10600 7650 0    69   ~ 14
+2
+Text Notes 8150 7650 0    50   ~ 0
+08/06/2020
+Wire Wire Line
+	5500 3250 5500 3350
 Wire Bus Line
 	5350 2250 5350 2750
@@
 Wire Bus Line
 	10750 4350 10750 5800
-Text Notes 7400 7500 0    69   Italic 14
-Homebrew Keyboard with Parallel Interface
-Text Notes 10600 7650 0    69   ~ 14
-2
-Text Notes 8150 7650 0    50   ~ 0
-08/06/2020
+Wire Wire Line
+	5500 3250 5550 3250
+Connection ~ 5500 3350
+Wire Wire Line
+	5200 2700 5200 5250
 $EndSCHEMATC
